Commit message: 将逆解计算器由KDL改为外置的TRAC-IK，将“接收下位机目标关节角度”改为“接收末端目标欧拉角”

File: src/engineer/urdf/engineer.urdf (robot description, URDF)
Before this commit: robot engineer, 12 links, 11 joints
Joints:
- joint joint6: axis 0 0 -1 -> 0 0 1; limit lower=-1.5 upper=0.15 effort=100 velocity=1.0 -> lower=-0.15 upper=1.5 effort=100 velocity=1.0
- joint joint7: axis 0 0 -1 -> 0 0 1; limit lower=-1.5 upper=0.0 effort=100 velocity=1.0 -> lower=0.0 upper=1.5 effort=100 velocity=1.0

Commit message: 修改了urdf轴和限位，新增笛卡尔直线规划

File: src/engineer/urdf/engineer.urdf (robot description, URDF)
Before this commit: robot engineer, 12 links, 11 joints
Joints:
- joint joint10: axis 0 0 1 -> 0 0 -1
- joint joint11: axis 0 0 1 -> 0 0 -1; limit lower=-3.1416 upper=3.1416 effort=100 velocity=1.0 -> lower=-3.909538 upper=1.570796 effort=100 velocity=1.0
- joint joint5: axis 0 0 -1 -> 0 0 1; limit lower=-3.1416 upper=3.1416 effort=100 velocity=1.0 -> lower=-2.012365 upper=3.886848 effort=100 velocity=1.0
- joint joint6: limit lower=-0.15 upper=1.5 effort=100 velocity=1.0 -> lower=0 upper=1.832596 effort=100 velocity=1.0
- joint joint7: limit lower=0.0 upper=1.5 effort=100 velocity=1.0 -> lower=0.017453 upper=2.583087 effort=100 velocity=1.0
- joint joint8: limit lower=-1.3 upper=0.1 effort=100 velocity=1.0 -> lower=-1.326450 upper=0.0 effort=100 velocity=1.0
- joint joint9: limit lower=-3.1416 upper=3.1416 effort=100 velocity=1.0 -> lower=-5.63683 upper=0.05236 effort=100 velocity=1.0
